File: Sdram_mister_deca/kicad/sdram_xs-SchDoc.sch (KiCad schematic (older format))
At the start: 24 parts, among them P1 Header 20X2, P8 Conn_02x23_Odd_Even

Commit message: update 2
Connections:
- net at P8.17 (Pin_17): no longer P1.11
Changed lines of the file:
@@
 	11700 2850 12500 2850
 Wire Wire Line
-	11700 2950 12500 2950
-Wire Wire Line
 	11700 3050 12500 3050
 Wire Wire Line
@@
 	13400 4500 13400 3850
 Connection ~ 13400 3850
-Wire Wire Line
-	6900 3850 7700 3850
-Wire Bus Line
-	7200 1750 7200 4450
-Wire Bus Line
-	9200 1750 9200 4350
-Wire Bus Line
-	6600 1750 6600 4050
-Wire Bus Line
-	4800 1750 4800 5150
 $Bitmap
 Pos 5750 8050
@@
 Data
 89 50 4E 47 0D 0A 1A 0A 00 00 00 0D 49 48 44 52 00 00 03 3D 00 00 02 8B 08 02 00 00 00 53 EE 71
-FE 00 00 00 03 73 42 49 54 08 08 08 DB E1 4F E0 00 00 00 09 70 48 59 73 00 00 0E C3 00 00 0E C3
-01 C7 6F A8 64 00 00 20 00 49 44 41 54 78 9C EC BD 79 78 5C D5 7D FF FF 3E E7 2E B3 8F A4 D1 6A
+FE 00 00 00 03 73 42 49 54 08 08 08 DB E1 4F E0 00 00 00 09 70 48 59 73 00 00 0E 74 00 00 0E 74
+01 6B 24 B3 D6 00 00 20 00 49 44 41 54 78 9C EC BD 79 78 5C D5 7D FF FF 3E E7 2E B3 8F A4 D1 6A
 59 B2 6C CB 1B 78 C3 06 EF 0B D8 10 CC 62 13 4A 5A 08 25 10 DA A4 4F DA A6 69 FA 10 B2 74 CD F7
 49 D3 A7 79 DA FE 92 D2 84 A6 6D 9A B4 C5 24 04 12 02 29 B8 66 F1 8A 37 6C 83 8D 6C CB B6 64 59
@@
 Text Notes 11550 8800 0    84   ~ 17
 FOR REFERENCE De10-Nano CONNECTOR
+Wire Wire Line
+	6900 3850 7700 3850
+Wire Bus Line
+	7200 1750 7200 4450
+Wire Bus Line
+	9200 1750 9200 4350
+Wire Bus Line
+	6600 1750 6600 4050
+Wire Bus Line
+	4800 1750 4800 5150
 $EndSCHEMATC
